Commit message: working intake

File: src/rift_description/urdf/parts/intake.xacro (robot description, xacro)
@@ -4,7 +4,7 @@
     <link name="intake_link">
         <visual>
-            <origin xyz="0 0 0" rpy="0 {pi}/2 0" />
+            <origin xyz="0 0 0" rpy="0 0 ${pi/2}" />
             <geometry>
-                <mesh filename="package://rift_description/meshes/RiftIntake.stl" scale="1 1 1" />
+                <mesh filename="package://rift_description/meshes/RiftIntake.stl" scale="0.001 0.001 0.001" />
             </geometry>
             <material name="blue"/>
@@ -31,16 +31,19 @@
             </geometry>
         </collision>
+        <xacro:inertial_box mass="0.5" x="0.575" y="0.127" z="0.22">
+            <origin xyz="0 0 0" rpy="0 0 0" />
+        </xacro:inertial_box>
     </link>
     <xacro:versaroller prefix="0" parent="intake_link">
-        <origin xyz="0 .10836 -0.008356" rpy="0 ${pi/2} 0" />
+        <origin xyz="${-0.10836 + 0.215} 0 ${-0.008356-0.005}" rpy="0 0 0" />
     </xacro:versaroller>
     <xacro:versaroller prefix="1" parent="intake_link">
-        <origin xyz="0.000201 0.045509 0.028214" rpy="0 ${pi/2} 0" />
+        <origin xyz=" ${-0.045509 + 0.215} 0.000201 ${0.028214-0.005}" rpy="0 0 0" />
     </xacro:versaroller>
     <xacro:versaroller prefix="2" parent="intake_link">
-        <origin xyz="-0.000036 0.088642 -0.08196" rpy="0 ${pi/2} 0" />
+        <origin xyz="${-0.088642 + 0.215} -0.000036  ${-0.08196-0.005}" rpy="0 0 0" />
     </xacro:versaroller>
     <xacro:versaroller prefix="3" parent="intake_link">
-        <origin xyz="-0.000053 0.0254 -0.045558" rpy="0 ${pi/2} 0" />
+        <origin xyz="${-0.0254 + 0.215} -0.000053 ${-0.045558-0.005}" rpy="0 0 0" />
     </xacro:versaroller>
     <joint name="intake_joint" type="fixed">

File: src/rift_description/urdf/parts/square_chassis.xacro (robot description, xacro)
@@ -19,5 +19,5 @@
         <origin xyz="0 0 ${chassis_height/2}" rpy="0 0 ${pi/2}" />
         <geometry>
-          <mesh filename="package://rift_description/meshes/SwerveChassis.stl" scale="0.001 0.001 0.001" />
+          <mesh filename="package://rift_description/meshes/RiftChassis.stl" scale="0.001 0.001 0.001" />
         </geometry>
         <material name="purple"/>

File: src/rift_description/urdf/parts/swerve_axle.xacro (robot description, xacro)
@@ -12,5 +12,5 @@
     <!-- NOTE: Pretty good **guesses**-->
     <xacro:property name="wheel_pos_y" value="0.022"/>
-    <xacro:property name="wheel_pos_z" value="0.063"/>
+    <xacro:property name="wheel_pos_z" value="0.025"/>
     <xacro:macro name="swerve_axle" params="prefix parent *origin">
         <link name="${prefix}_axle_link">
@@ -35,5 +35,5 @@
         <link name="${prefix}_wheel_link">
             <visual>
-                <origin xyz="0 ${wheel_pos_y} 0" rpy="${pi / 2} 0 ${pi / 4}" />
+                <origin xyz="0 0 0" rpy="${pi / 2} 0 ${pi/2}" />
                 <geometry>
                     <mesh filename="package://rift_description/meshes/SwerveWheel.stl" scale="0.001 0.001 0.001" />

File: src/rift_description/urdf/parts/versaroller.xacro (robot description, xacro)
@@ -4,4 +4,11 @@
     <xacro:macro name="versaroller" params="prefix parent *origin">
     <link name="intake_rollerbar_${prefix}_link">
+        <visual>
+            <origin xyz="0 0 0" rpy="0 ${pi/2} ${pi/2}" />
+            <geometry>
+                <cylinder length="0.575" radius="0.016"/>
+            </geometry>
+            <material name="yellow" />
+        </visual>
         <collision>
             <geometry>

File: src/rift_description/urdf/robots/rift.urdf.xacro (robot description, xacro)
@@ -22,5 +22,5 @@
   <!-- Axle Position Variables -->
   <xacro:property name="axle_pos" value="0.261523" />
-  <xacro:property name="axle_pos_z" value="${69.056 / 1000}" />
+  <xacro:property name="axle_pos_z" value="${39.056 / 1000}" />
   <xacro:property name="elevator_middle_distance" value = ".457" />
   <xacro:property name= "chassis_side_width" value = ".0254" />
@@ -33,9 +33,9 @@
   <link name="base_link">
   <!-- Set mass to 0 and give a valid inertia tensor of 0 -->
-    <inertial>
+    <!-- <inertial>
       <mass value="0.0"/>
       <origin xyz="0 0 0" rpy="0 0 0"/>
       <inertia ixx="0.0" ixy="0.0" ixz="0.0" iyy="0.0" iyz="0.0" izz="0.0"/>
-    </inertial>
+    </inertial> -->
   </link>
   <xacro:square_chassis prefix="swerve" parent="base_link">
@@ -43,16 +43,16 @@
   </xacro:square_chassis>
   <!-- Arm -->
-  <xacro:arm parent="base_link">
+  <!-- <xacro:arm parent="base_link">
     <origin xyz="0 0 0" rpy="0 0 0" />
-  </xacro:arm>
+  </xacro:arm> -->
   <!-- Intake -->
   <xacro:intake parent="swerve_chassis_link">
-    <origin xyz="0.46 0 0.09" rpy="0 0 ${pi/2}" />
+    <origin xyz="0.24 0 0.09" rpy="0 0 0" />
   </xacro:intake>
-  <!-- Shooter -->
+  <!-- Shooter
   <xacro:shooter prefix="shooter" parent="base_link">
-    <!-- <origin xyz="0 0 0" rpy="0 0 0" /> -->
-    <origin xyz="0.25 0 .33" rpy="0 ${-pi/6} 0" /> <!-- Made up values for shooter location & rotation. Change later. -->
-  </xacro:shooter>
+    <origin xyz="0 0 0" rpy="0 0 0" />
+    <origin xyz="0.25 0 .33" rpy="0 ${-pi/6} 0" /> Made up values for shooter location & rotation. Change later.
+  </xacro:shooter> -->
   <!-- Drive Train -->
   <xacro:swerve_axle prefix="front_left" parent="swerve_chassis_link">
