Commit message: made urdf look like robot

File: src/rift_description/urdf/parts/arm.xacro (robot description, xacro)
@@ -2,62 +2,63 @@
 <robot xmlns:xacro="http://www.ros.org/wiki/xacro">
     <!-- Arm Properties -->
-    <xacro:property name="arm_bar_length" value="0.0508" />
-    <xacro:property name="arm_bar_width" value="0.0254" />
-    <xacro:property name="arm_bar_height" value="0.445" />
-    <xacro:property name="arm_mount_weight" value="0.419029447872" />
-    <xacro:property name="arm_mount_length" value="0.0508" />
-    <xacro:property name="arm_mount_width" value="0.356" />
-    <xacro:property name="arm_mount_height" value="0.0254" />
-    <xacro:property name="arm_mount_weight" value="0.7589489" />
+    <xacro:property name="arm_bar_height" value="0.0508" />
+    <xacro:property name="arm_bar_width" value="0.30" />
+    <xacro:property name="arm_bar_length" value="0.5" />
+    <xacro:property name="arm_bar_weight" value="0.419029447872" />
+    <xacro:property name="arm_mount_weight" value="7589489" /> <!-- This is a guess -->
+    <xacro:property name="arm_mount_length" value="0.25" />
+    <xacro:property name="arm_mount_width" value="0.25" />
+    <xacro:property name="arm_mount_height" value="0.25" />
     <xacro:macro name="arm" params="parent *origin">
-        <!-- Left Bar Arm -->
-        <link name="left_bar_link">
+        <link name="arm_mount_link">
             <visual>
-                <origin xyz="${-arm_mount_width/2} 0 0" rpy="0 ${pi/2} ${pi/2}"/>
-                <geometry>
-                <!-- Mesh File doesnt work -->
-                    <mesh filename="package://rift_description/meshes/ArmPart.stl" scale="1 1 1"/>
-                    <box size="${arm_bar_length} ${arm_bar_width} ${arm_bar_height}"/>
-                </geometry>
-                <material name="red"/>
+                <origin xyz="0 0 0" rpy="0 0 ${pi/2}"/>
+                    <geometry>
+                        <mesh filename="package://rift_description/meshes/RiftSuperstructure.stl" scale="0.001 0.001 0.001"/>
+                    </geometry>
+                <material name="yellow"/>
             </visual>
             <collision>
+                <origin xyz="0 0 0" rpy="0 0 0"/>
+                <geometry>
+                    <box size="${arm_mount_length} ${arm_mount_width} ${arm_mount_height}"/>
+                </geometry>
             </collision>
+            <xacro:inertial_box mass="${arm_mount_weight}" x="${arm_mount_length}" y="${arm_mount_width}" z="${arm_mount_height}">
+                <origin xyz="0 0 0" rpy="0 0 0"/>
+            </xacro:inertial_box>
+            <!-- <xacro:inertial_box mass="0.5" xyz="0 0 0" size="0.5 0.5 0.5"/> -->
         </link>
-        <!-- Right Bar Arm -->
-        <link name="right_bar_link">
+        <link name="arm_bar_link">
+            <xacro:inertial_box mass="${arm_mount_weight}" x="${arm_mount_length}" y="${arm_mount_width}" z="${arm_mount_height}">
+                <origin xyz="0 0 0" rpy="0 0 0"/>
+            </xacro:inertial_box>
             <visual>
-            <origin xyz="${arm_mount_width/2} 0 0" rpy="0 ${pi/2} ${pi/2}"/>
+                <origin xyz="0.18 0 0" rpy="0 0 ${pi/2}"/>
                 <geometry>
-                <!-- Mesh File Does Not Work -->
-                    <mesh filename="package://rift_description/meshes/ArmPart.stl" scale="1 1 1"/>
-                    <box size="${arm_bar_length} ${arm_bar_width} ${arm_bar_height}"/>
-                </geometry>
-                <material name="red"/>
-            </visual>
-            <collision>
-            </collision>
-        </link>
-        <!-- Arm Mount -->
-        <link name="arm_mount_link">
-            <visual>
-                <origin xyz="0 ${arm_bar_height/2} 0" rpy="${pi/2} ${pi/2} 0"/>
-                <geometry>
-                <!-- Mesh File Does not Work -->
-                    <mesh filename="package://rift_description/meshes/ShooterMount.stl" scale="1 1 1"/>
-                    <box size="${arm_mount_length} ${arm_mount_width} ${arm_mount_height}"/>
+                    <mesh filename="package://rift_description/meshes/RiftShooterArm.stl" scale="0.001 0.001 0.001"/>
                 </geometry>
                 <material name="yellow"/>
             </visual>
             <collision>
+                <origin xyz="0.18 0 0" rpy="0 -${pi/60} 0"/>
+                <geometry>
+                    <box size="${arm_bar_length} ${arm_bar_width} ${arm_bar_height}"/>
+                </geometry>
             </collision>
         </link>
         <joint name="arm_mount_joint" type="fixed">
-            <origin xyz = "0 0 .2" rpy = "0 0 0"/>
             <parent link="${parent}"/>
             <child link="arm_mount_link"/>
             <xacro:insert_block name="origin" />
         </joint>
-        <joint name="left_bar_joint" type="fixed">
+        <joint name="arm_bar_joint" type="revolute">
+            <origin xyz="-0.12 0 0.13" rpy="0 0 0"/>
+            <parent link="arm_mount_link"/>
+            <child link="arm_bar_link"/>
+            <limit effort="100" velocity="100" lower="0" upper="1.57"/>
+            <xacro:insert_block name="origin" />
+        </joint>
+        <!-- <joint name="left_bar_joint" type="fixed">
             <origin xyz = "0 0 0" rpy = "0 0 0"/>
             <parent link="arm_mount_link"/>
@@ -70,5 +71,5 @@
             <child link="right_bar_link"/>
             <xacro:insert_block name="origin" />
-        </joint>
+        </joint> -->
     </xacro:macro>
 </robot>

File: src/rift_description/urdf/parts/intake.xacro (robot description, xacro)
@@ -12,12 +12,12 @@
         <!-- Front plate collision -->
         <collision>
-            <origin xyz="0 ${0.0254/2} 0" rpy="0 0 0" />
+            <origin xyz="0.21 0 0" rpy="0 0 ${pi/2}" />
             <geometry>
-                <box size="0.575 0.0254 0.102" />
+                <box size="0.64 0.0254 0.102" />
             </geometry>
         </collision>
         <!-- +Y side collision -->
         <collision>
-            <origin xyz="${0.575/2+0.038/2} 0.065 0.007" rpy="0 0 0" />
+            <origin xyz="0.12 ${0.575/2+0.038/2} 0.007" rpy="0 0 ${pi/2}" />
             <geometry>
                 <box size="0.038 0.127 0.22" />
@@ -26,5 +26,5 @@
         <!-- -Y side collision -->
         <collision>
-            <origin xyz="${-0.575/2-0.038/2} 0.065 0.007" rpy="0 0 0" />
+            <origin xyz="0.12 ${-0.575/2-0.038/2} 0.007" rpy="0 0 ${pi/2}" />
             <geometry>
                 <box size="0.038 0.127 0.22" />

File: src/rift_description/urdf/parts/shooter.xacro (robot description, xacro)
@@ -17,15 +17,18 @@
     <xacro:property name="sidepanel_height" value="0.426" />
     <xacro:property name="sidepanel_y_offset" value="0.186088" />
-    <xacro:property name="wheel_length" value="0.363538" />
-    <xacro:property name="wheel_radius" value="0.0505" />
-    <xacro:property name="wheel_x_offset" value="0.08" /> <!-- This is a guess -->
-    <xacro:property name="wheel_z_offset" value="0.156" /> <!-- This is a guess -->
-    <xacro:property name="wheel_mass" value="${0.11566605*4}" /> <!--not the most accurate, but issok-->
-    <xacro:macro name="shooter" params="prefix parent *origin">
-        <link name="${prefix}_link">
+    <xacro:property name="shooter_wheel_length" value="0.363538" />
+    <xacro:property name="shooter_wheel_radius" value="0.0505" />
+    <xacro:property name="shooter_wheel_x_offset" value="0.1" /> <!-- This is a guess -->
+    <xacro:property name="shooter_wheel_y_offset" value="0.05" /> <!-- This is a guess -->
+    <xacro:property name="shooter_wheel_z_offset" value="0.17" /> <!-- This is a guess -->
+    <xacro:property name="intake_roller_radius" value="0.01" /> <!-- This is a guess -->
+    <xacro:property name="intake_roller_mass" value="${0.11566605}" /> <!-- This is a guess -->
+    <xacro:property name="shooter_wheel_mass" value="${0.11566605*4}" /> <!--not the most accurate, but issok-->
+    <xacro:macro name="shooter" params="parent *origin">
+        <link name="shooter_link">
             <visual>
-                <origin xyz="${mesh_x_offset} 0 ${mesh_z_offset}" rpy="0 ${pi/2} 0" />
+                <origin xyz="0 0 0" rpy="${pi} -${pi/2} -${pi/2}" />
                 <geometry>
-                    <mesh filename="package://rift_description/meshes/RiftShooter.stl" scale="1 1 1" />
+                    <mesh filename="package://rift_description/meshes/RiftShooter.stl" scale="0.001 0.001 0.001" />
                 </geometry>
                 <material name="red" />
@@ -38,5 +41,5 @@
             </collision>
             <collision>
-                <origin xyz="0 ${-(sidepanel_y_offset - sidepanel_width/2)} 0" rpy="0 0 0" />
+                <origin xyz="0 ${-(sidepanel_y_offset - sidepanel_width/2)} 0" rpy="0 0 0"/>
                 <geometry>
                     <box size="${sidepanel_length} ${sidepanel_width} ${sidepanel_height}" />
@@ -44,85 +47,108 @@
             </collision>
         </link>
-        <link name="${prefix}_wheels_forward_link">
+        <link name="shooter_wheels_forward_link">
+            <visual>
+                <origin xyz="0 0 0" rpy="${pi/2} 0 ${pi/2}" />
+                <geometry>
+                    <mesh filename="package://rift_description/meshes/RiftShooterRoller.stl" scale="0.001 0.001 0.001" />
+                </geometry>
+                <material name="green" />
+            </visual>
             <collision>
                 <origin xyz="0 0 0" rpy="${pi / 2} 0 0" />
                 <geometry>
-                    <cylinder length="${wheel_length}" radius="${wheel_radius}" />
+                    <cylinder length="${shooter_wheel_length}" radius="${shooter_wheel_radius}" />
                 </geometry>
             </collision>
             <!-- Pretty sure something is wrong with this, but I don't know what... -->
-            <xacro:inertial_cylinder mass="${wheel_mass}" radius="${wheel_radius}" length="${wheel_length}">
+            <xacro:inertial_cylinder mass="${shooter_wheel_mass}" radius="${shooter_wheel_radius}" length="${shooter_wheel_length}">
                 <origin xyz="0 0 0" rpy="${pi / 2} 0 0" />
             </xacro:inertial_cylinder>
         </link>
-        <link name="${prefix}_wheels_backward_link">
+        <link name="shooter_wheels_backward_link">
+            <visual>
+                <origin xyz="0 0 0" rpy="${pi/2} 0 ${pi/2}" />
+                <geometry>
+                    <mesh filename="package://rift_description/meshes/RiftShooterRoller.stl" scale="0.001 0.001 0.001" />
+                </geometry>
+                <material name="green" />
+            </visual>
             <collision>
                 <origin xyz="0 0 0" rpy="${pi / 2} 0 0" />
                 <geometry>
-                    <cylinder length="${wheel_length}" radius="${wheel_radius}" />
+                    <cylinder length="${shooter_wheel_length}" radius="${shooter_wheel_radius}" />
                 </geometry>
             </collision>
             <!-- Pretty sure something is wrong with this, but I don't know what... -->
-            <xacro:inertial_cylinder mass="${wheel_mass}" radius="${wheel_radius}" length="${wheel_length}">
+            <xacro:inertial_cylinder mass="${shooter_wheel_mass}" radius="${shooter_wheel_radius}" length="${shooter_wheel_length}">
                 <origin xyz="0 0 0" rpy="${pi / 2} 0 0" />
             </xacro:inertial_cylinder>
         </link>
-        <!-- <link name="${prefix}_backPanel_link">
-            <xacro:inertial_box mass="0.02" x="${back_panel_length}" y="${panel_height}"
-                z="${back_panel_thick}">
-                <origin xyz="0 0 0" rpy="0 0 0" />
-            </xacro:inertial_box>
-            <visual>
-                <origin xyz="0 0 0" rpy="0 0 0" />
-                <geometry>
-                    <box size="${back_panel_width} ${panel_height} ${back_panel_thick}" />
-                </geometry>
-                <material name="red" />
-            </visual>
-            <collision>
-                <origin xyz="0 0 0" rpy="0 0 0" />
-                <geometry>
-                    <box size="${back_panel_width} ${panel_height} ${back_panel_thick}" />
-                </geometry>
-            </collision>
-        </link>
-        <link name="${prefix}_frontPanel_link">
-            <xacro:inertial_box mass="0.02" x="${back_panel_length}" y="${panel_height}"
-                z="${back_panel_thick}">
-                <origin xyz="0 0 0" rpy="0 0 0" />
-            </xacro:inertial_box>
-            <visual>
-                <origin xyz="0 0 0" rpy="0 0 0" />
-                <geometry>
-                    <box size="${back_panel_width} ${panel_height} ${back_panel_thick}" />
-                </geometry>
-                <material name="red" />
-            </visual>
-            <collision>
-                <origin xyz="0 0 0" rpy="0 0 0" />
-                <geometry>
-                    <box size="${back_panel_width} ${panel_height} ${back_panel_thick}" />
-                </geometry>
-            </collision>
-        </link> -->
-        <joint name="${prefix}_joint" type="fixed">
+        <xacro:macro name="shooter_intake_roller" params="number">
+            <link name="shooter_intake_roller_${number}_link">
+                <visual>
+                    <origin xyz="0 0 0" rpy="${pi/2} 0 ${pi/2}" />
+                    <geometry>
+                        <mesh filename="package://rift_description/meshes/RiftShooterIntakeRoller.stl" scale="0.001 0.001 0.001" />
+                    </geometry>
+                    <material name="green" />
+                </visual>
+                <collision>
+                    <origin xyz="0 0 0" rpy="${pi / 2} 0 0" />
+                    <geometry>
+                        <cylinder length="${shooter_wheel_length}" radius="${intake_roller_radius}" />
+                    </geometry>
+                </collision>
+                <!-- Pretty sure something is wrong with this, but I don't know what... -->
+                <xacro:inertial_cylinder mass="${intake_roller_mass}" radius="${intake_roller_radius}" length="${shooter_wheel_length}">
+                    <origin xyz="0 0 0" rpy="${pi / 2} 0 0" />
+                </xacro:inertial_cylinder>
+            </link>
+            <joint name="shooter_intake_roller_${number}_joint" type="continuous">
+                <!-- <xacro:if value="${position == 'front'}">
+                    <origin xyz="${-shooter_wheel_x_offset} 0 ${shooter_wheel_z_offset}" rpy="0 0 0" />
+                </xacro:if> -->
+                <origin xyz="${0.02 + ((number % 5) * 0.035) - (number - (number % 5))/5 * 0.065 } 0 ${0.07 - (number % 5 ) * 0.054 - (number - (number % 5))/5 * 0.042}" rpy="0 0 0" />
+                <parent link="shooter_link" />
+                <child link="shooter_intake_roller_${number}_link" />
+                <axis xyz="0 1 0" />
+            </joint>
+        </xacro:macro>
+        <joint name="shooter_joint" type="fixed">
             <parent link="${parent}" />
-            <child link="${prefix}_link" />
+            <child link="shooter_link" />
             <xacro:insert_block name="origin" />
         </joint>
-        <joint name="${prefix}_wheels_forward_joint" type="fixed">
-            <origin xyz="${wheel_x_offset} 0 ${wheel_z_offset}" rpy="0 0 0" />
-            <parent link="${prefix}_link" />
-            <child link="${prefix}_wheels_forward_link" />
+        <joint name="shooter_wheels_forward_joint" type="continuous">
+            <origin xyz="-0.008 ${shooter_wheel_y_offset} ${shooter_wheel_z_offset-0.012}" rpy="0 0 0" />
+            <parent link="shooter_link" />
+            <child link="shooter_wheels_forward_link" />
             <axis xyz="0 1 0" />
             <limit effort="100" lower="-1" upper="1" velocity="2" />
         </joint>
-        <joint name="${prefix}_wheels_backward_joint" type="fixed">
-            <origin xyz="${-(wheel_x_offset - wheel_radius/2)} 0 ${wheel_z_offset}" rpy="0 0 0" />
-            <parent link="${prefix}_link" />
-            <child link="${prefix}_wheels_backward_link" />
+        <joint name="shooter_wheels_backward_joint" type="continuous">
+            <origin xyz="${-(shooter_wheel_x_offset) - shooter_wheel_radius/2} ${shooter_wheel_y_offset} ${shooter_wheel_z_offset/2}" rpy="0 0 0" />
+            <parent link="shooter_link" />
+            <child link="shooter_wheels_backward_link" />
             <axis xyz="0 1 0" />
             <limit effort="100" lower="-1" upper="1" velocity="2" />
         </joint>
+        <xacro:shooter_intake_roller number="1"/>
+        <xacro:shooter_intake_roller number="2"/>
+        <xacro:shooter_intake_roller number="3"/>
+        <xacro:shooter_intake_roller number="4"/>
+        <xacro:shooter_intake_roller number="5"/>
+        <xacro:shooter_intake_roller number="6"/>
+        <xacro:shooter_intake_roller number="7"/>
+        <xacro:shooter_intake_roller number="8"/>
+        <xacro:shooter_intake_roller number="9"/>
+        <xacro:shooter_intake_roller number="10"/>
+        <!-- <joint>
+            <origin xyz="0 0 0" rpy="0 0 0" />
+            <parent link="shooter_link" />
+            <child link="shooter_intake_roller_link" />
+            <axis xyz="0 1 0" />
+            <limit effort="100" lower="-1" upper="1" velocity="2" />
+        </joint> -->
     </xacro:macro>
 </robot>

File: src/rift_description/urdf/parts/versaroller.xacro (robot description, xacro)
@@ -2,4 +2,7 @@
 <robot xmlns:xacro="http://www.ros.org/wiki/xacro">
     <!-- I made this file just because I felt that having it four times in the intake was a *bad* idea. Feel free to give better ideas. -->
+    <xacro:property name="rollerbar_length" value="0.575" />
+    <xacro:property name="rollerbar_radius" value="0.016" />
+    <xacro:property name="rollerbar_mass" value="0.5" />
     <xacro:macro name="versaroller" params="prefix parent *origin">
     <link name="intake_rollerbar_${prefix}_link">
@@ -7,9 +10,10 @@
             <origin xyz="0 0 0" rpy="0 ${pi/2} ${pi/2}" />
             <geometry>
-                <cylinder length="0.575" radius="0.016"/>
+                <cylinder length="${rollerbar_length}" radius="${rollerbar_radius}"/>
             </geometry>
             <material name="yellow" />
         </visual>
         <collision>
+            <origin xyz="0 0 0" rpy="0 ${pi/2} ${pi/2}" />
             <geometry>
                 <cylinder length="0.575" radius="0.016"/>
@@ -17,4 +21,7 @@
             <!-- <material name="ghost" /> -->
         </collision>
+        <xacro:inertial_cylinder mass="${rollerbar_mass}" radius="${rollerbar_radius}" length="${rollerbar_length}">
+            <origin xyz="0 0 0" rpy="0 0 0" />
+        </xacro:inertial_cylinder>
     </link>
     <joint name="intake_rollerbar_${prefix}_joint" type="continuous">
